File: hardware/pcb/kicad/WALKIN_PIR_IF.kicad_pcb (KiCad board)
At the start: 2 copper layers, 67.1 x 42.9 mm, 22 parts, among them J1 Battery Terminal, J2 XWA11V Terminal, J3 Probe Terminal, Q1 AO3401A, U1 AQY212EH

Commit message: fab diagram and 3d render
Other:
- board text added: "⌀3.2"
